File: KiCad/ZX21/ZX21.sch (KiCad schematic (older format))
At the start: 85 parts, among them IC1 ULA 2C210E, IC101 555, IC2 AT28C256, IC3 Z80A, IC4 62256, J1 Jack-DC, J203 Conn_01x03, J204 Conn_01x03, X1 3.5MHz

Commit message: Add Gate
Parts:
- added C105: 100N, Capacitors_SMD:C_0603_HandSoldering, symbol device:C
- added IC102: 74HCT00, Housings_SOIC:SOIC-14_3.9x8.7mm_Pitch1.27mm, symbol Logic_74xx:74HCT00
- added J2: Conn_01x02, Pin_Headers:Pin_Header_Straight_1x02_Pitch2.54mm, symbol Connector:Conn_01x02
- added R105: 4K7, Resistors_SMD:R_0603_HandSoldering, symbol device:R
Connections:
- wire segments 416 -> 434
Changed lines of the file:
@@
 Wire Wire Line
 	5950 4725 5950 6125
-Connection ~ 7100 1725
-Connection ~ 7200 1825
-Connection ~ 7300 1925
-Connection ~ 7400 2025
 Connection ~ 7500 2125
 Connection ~ 7600 2225
@@
 Wire Wire Line
 	7000 1625 7000 3125
-Wire Wire Line
-	7100 1725 7100 3125
-Wire Wire Line
-	7200 1825 7200 3125
-Wire Wire Line
-	7300 1925 7300 3125
-Wire Wire Line
-	7400 2025 7400 3125
 Wire Wire Line
 	7500 2125 7500 3125
@@
 	5750 625  5750 1125
 Wire Wire Line
-	6150 1725 7100 1725
-Wire Wire Line
-	6150 1825 7200 1825
-Wire Wire Line
-	6150 1925 7300 1925
-Wire Wire Line
-	6150 2025 7400 2025
-Wire Wire Line
 	6150 2125 7500 2125
 Wire Wire Line
@@
 Wire Wire Line
 	7500 2125 9050 2125
-Wire Wire Line
-	7400 2025 9100 2025
-Wire Wire Line
-	7300 1925 9150 1925
-Wire Wire Line
-	7200 1825 9200 1825
-Wire Wire Line
-	7100 1725 9250 1725
 Wire Wire Line
 	7000 1625 9300 1625
@@
 ROW8
 $Sheet
-S 7775 775  1100 325
+S 9650 3525 1100 325
 U 632617C4
 F0 "Extras" 50
@@
 Wire Wire Line
 	4750 2475 4750 2425
+Wire Wire Line
+	6150 1725 9250 1725
+Wire Wire Line
+	6150 1825 9200 1825
+Wire Wire Line
+	6150 1925 9150 1925
+Wire Wire Line
+	6150 2025 9100 2025
+$Comp
+L Logic_74xx:74HCT00 IC102
+U 1 1 5FD1E154
+P 7100 1025
+F 0 "IC102" V 7075 900 50  0000 L CNN
+F 1 "74HCT00" V 7375 2525 50  0001 L CNN
+F 2 "Housings_SOIC:SOIC-14_3.9x8.7mm_Pitch1.27mm" H 7100 1025 50  0001 C CNN
+F 3 "http://www.ti.com/lit/gpn/sn74hct00" H 7100 1025 50  0001 C CNN
+	1    7100 1025
+	0    1    1    0
+$EndComp
+$Comp
+L Logic_74xx:74HCT00 IC102
+U 2 1 5FD21B16
+P 7500 1025
+F 0 "IC102" V 7475 875 50  0000 L CNN
+F 1 "74HCT00" H 7600 1175 50  0001 L CNN
+F 2 "Housings_SOIC:SOIC-14_3.9x8.7mm_Pitch1.27mm" H 7500 1025 50  0001 C CNN
+F 3 "http://www.ti.com/lit/gpn/sn74hct00" H 7500 1025 50  0001 C CNN
+	2    7500 1025
+	0    1    1    0
+$EndComp
+$Comp
+L Logic_74xx:74HCT00 IC102
+U 3 1 5FD24E41
+P 7900 1025
+F 0 "IC102" V 7875 900 50  0000 L CNN
+F 1 "74HCT00" V 7945 1213 50  0001 L CNN
+F 2 "Housings_SOIC:SOIC-14_3.9x8.7mm_Pitch1.27mm" H 7900 1025 50  0001 C CNN
+F 3 "http://www.ti.com/lit/gpn/sn74hct00" H 7900 1025 50  0001 C CNN
+	3    7900 1025
+	0    1    1    0
+$EndComp
+$Comp
+L Logic_74xx:74HCT00 IC102
+U 4 1 5FD25FC1
+P 8275 1025
+F 0 "IC102" V 8250 900 50  0000 L CNN
+F 1 "74HCT00" V 8450 1150 50  0000 L CNN
+F 2 "Housings_SOIC:SOIC-14_3.9x8.7mm_Pitch1.27mm" H 8275 1025 50  0001 C CNN
+F 3 "http://www.ti.com/lit/gpn/sn74hct00" H 8275 1025 50  0001 C CNN
+	4    8275 1025
+	0    1    1    0
+$EndComp
+Wire Wire Line
+	7100 3125 7100 1325
+Wire Wire Line
+	7200 3125 7200 1325
+Wire Wire Line
+	7200 1325 7500 1325
+Wire Wire Line
+	7300 3125 7300 1375
+Wire Wire Line
+	7300 1375 7900 1375
+Wire Wire Line
+	7900 1375 7900 1325
+Wire Wire Line
+	8275 1325 8275 1450
+Wire Wire Line
+	8275 1450 7400 1450
+Wire Wire Line
+	7400 1450 7400 3125
+Text GLabel 7000 725  1    50   Input ~ 0
+A13
+Text GLabel 7400 725  1    50   Input ~ 0
+A12
+Text GLabel 7800 725  1    50   Input ~ 0
+A11
+Text GLabel 8175 725  1    50   Input ~ 0
+A10
+Wire Wire Line
+	7200 725  7200 500
+Wire Wire Line
+	7200 500  7600 500
+Wire Wire Line
+	8375 500  8375 575
+Wire Wire Line
+	8000 725  8000 500
+Connection ~ 8000 500
+Wire Wire Line
+	8000 500  8375 500
+Wire Wire Line
+	7600 725  7600 500
+Connection ~ 7600 500
+Wire Wire Line
+	7600 500  8000 500
+$Comp
+L Connector:Conn_01x02 J2
+U 1 1 5FEF73ED
+P 8800 675
+F 0 "J2" H 8880 667 50  0000 L CNN
+F 1 "Conn_01x02" H 8880 576 50  0001 L CNN
+F 2 "Pin_Headers:Pin_Header_Straight_1x02_Pitch2.54mm" H 8800 675 50  0001 C CNN
+F 3 "~" H 8800 675 50  0001 C CNN
+	1    8800 675
+	1    0    0    -1
+$EndComp
+$Comp
+L power:GND #PWR0154
+U 1 1 5FF29BAB
+P 9175 900
+F 0 "#PWR0154" H 9175 650 50  0001 C CNN
+F 1 "GND" V 9275 925 50  0000 R CNN
+F 2 "" H 9175 900 50  0001 C CNN
+F 3 "" H 9175 900 50  0001 C CNN
+	1    9175 900
+	1    0    0    -1
+$EndComp
+$Comp
+L device:R R105
+U 1 1 5FF3AB29
+P 8525 575
+F 0 "R105" V 8525 575 50  0000 C CNN
+F 1 "4K7" V 8575 375 50  0000 C CNN
+F 2 "Resistors_SMD:R_0603_HandSoldering" V 8455 575 50  0001 C CNN
+F 3 "" H 8525 575 50  0001 C CNN
+	1    8525 575
+	0    -1   -1   0
+$EndComp
+Connection ~ 8375 575
+$Comp
+L power:+5V #PWR0155
+U 1 1 5FF3B39F
+P 9275 575
+F 0 "#PWR0155" H 9275 425 50  0001 C CNN
+F 1 "+5V" V 9225 625 50  0000 L CNN
+F 2 "" H 9275 575 50  0001 C CNN
+F 3 "" H 9275 575 50  0001 C CNN
+	1    9275 575
+	0    1    1    0
+$EndComp
+Wire Wire Line
+	8375 575  8375 675
+$Comp
+L device:C C105
+U 1 1 6000A744
+P 9175 750
+F 0 "C105" H 9290 796 50  0000 L CNN
+F 1 "100N" H 9290 705 50  0000 L CNN
+F 2 "Capacitors_SMD:C_0603_HandSoldering" H 9213 600 50  0001 C CNN
+F 3 "" H 9175 750 50  0001 C CNN
+	1    9175 750
+	1    0    0    -1
+$EndComp
+Wire Wire Line
+	23900 -12450 25675 -12450
+Wire Wire Line
+	25675 -12450 25675 -13400
+Wire Wire Line
+	8675 575  9175 575
+Wire Wire Line
+	9175 575  9175 600
+Connection ~ 9175 575
+Wire Wire Line
+	9175 575  9275 575
+Wire Wire Line
+	9175 900  8600 900
+Wire Wire Line
+	8600 900  8600 775
+Connection ~ 9175 900
+Wire Wire Line
+	8600 675  8375 675
+Connection ~ 8375 675
+Wire Wire Line
+	8375 675  8375 725
 $EndSCHEMATC
