File: KiCad/ZX21/ZX21.sch (KiCad schematic (older format))
At the start: 89 parts, among them IC1 ULA 2C210E, IC101 555, IC102 74HCT00, IC2 AT28C256, IC3 Z80A, IC4 62256, J1 Jack-DC, J2 Conn_01x02, J203 Conn_01x03, J204 Conn_01x03, X1 3.5MHz

Commit message: Part way through routing
Changed lines of the file:
@@
 	3750 4575 8300 4575
-Wire Wire Line
-	3650 4625 8400 4625
 Wire Wire Line
 	4450 1550 4375 1550
@@
 F 3 "http://www.ti.com/lit/gpn/sn74hct00" H 7900 1025 50  0001 C CNN
 	3    7900 1025
-	0    1    1    0
+	0    -1   1    0
 $EndComp
 $Comp
@@
 U 4 1 5FD25FC1
 P 8275 1025
-F 0 "IC102" V 8250 900 50  0000 L CNN
-F 1 "74HCT00" V 8450 1150 50  0000 L CNN
+F 0 "IC102" V 8250 875 50  0000 L CNN
+F 1 "74HCT00" V 8450 625 50  0000 L CNN
 F 2 "Housings_SOIC:SOIC-14_3.9x8.7mm_Pitch1.27mm" H 8275 1025 50  0001 C CNN
 F 3 "http://www.ti.com/lit/gpn/sn74hct00" H 8275 1025 50  0001 C CNN
 	4    8275 1025
-	0    1    1    0
+	0    -1   1    0
 $EndComp
 Wire Wire Line
@@
 Wire Wire Line
 	8375 675  8375 725
+Wire Wire Line
+	3650 4625 8400 4625
+$Comp
+L power:+5V #PWR0144
+U 1 1 5FD3AC5D
+P 5200 4675
+F 0 "#PWR0144" H 5200 4525 50  0001 C CNN
+F 1 "+5V" H 5215 4848 50  0000 C CNN
+F 2 "" H 5200 4675 50  0001 C CNN
+F 3 "" H 5200 4675 50  0001 C CNN
+	1    5200 4675
+	-1   0    0    1
+$EndComp
+$Comp
+L power:GND #PWR0157
+U 1 1 5FD3E8CA
+P 5200 6075
+F 0 "#PWR0157" H 5200 5825 50  0001 C CNN
+F 1 "GND" H 5205 5902 50  0000 C CNN
+F 2 "" H 5200 6075 50  0001 C CNN
+F 3 "" H 5200 6075 50  0001 C CNN
+	1    5200 6075
+	-1   0    0    1
+$EndComp
 $EndSCHEMATC

Commit message: Even more routing
Parts:
- added unit 5 of IC102
Connections:
- wire segments 434 -> 439
Other:
- moved on the sheet: C105, EDGE1
Changed lines of the file:
@@
 	1300 5725 1725 5725
 Text GLabel 6150 3775 2    50   Input ~ 0
-BUSAK
+BUSRQ
 Text GLabel 6150 3875 2    50   Input ~ 0
 RFSH
@@
 Text GLabel 3850 5425 0    50   Input ~ 0
 D0'
-Text Notes 10025 3300 0    50   ~ 0
+Text Notes 10000 4275 0    50   ~ 0
 A Top B Bottom
-Text GLabel 9850 3100 0    50   Input ~ 0
+Text GLabel 9825 4075 0    50   Input ~ 0
 RFSH
-Text GLabel 9850 3000 0    50   Input ~ 0
+Text GLabel 9825 3975 0    50   Input ~ 0
 MI
-Text GLabel 9850 2900 0    50   Input ~ 0
+Text GLabel 9825 3875 0    50   Input ~ 0
 RESET
-Text GLabel 9850 2800 0    50   Input ~ 0
+Text GLabel 9825 3775 0    50   Input ~ 0
 BUSRQ
-Text GLabel 9850 2700 0    50   Input ~ 0
+Text GLabel 9825 3675 0    50   Input ~ 0
 WAIT
-Text GLabel 9850 2600 0    50   Input ~ 0
+Text GLabel 9825 3575 0    50   Input ~ 0
 BUSAK
-Text GLabel 10750 3100 2    50   Input ~ 0
+Text GLabel 10725 4075 2    50   Input ~ 0
 ROM_CS
-Text GLabel 10750 3000 2    50   Input ~ 0
+Text GLabel 10725 3975 2    50   Input ~ 0
 A4
-Text GLabel 10750 2900 2    50   Input ~ 0
+Text GLabel 10725 3875 2    50   Input ~ 0
 A5
-Text GLabel 10750 2800 2    50   Input ~ 0
+Text GLabel 10725 3775 2    50   Input ~ 0
 A6
-Text GLabel 10750 2700 2    50   Input ~ 0
+Text GLabel 10725 3675 2    50   Input ~ 0
 A7
-Text GLabel 10750 2600 2    50   Input ~ 0
+Text GLabel 10725 3575 2    50   Input ~ 0
 A8
-Text GLabel 10750 2500 2    50   Input ~ 0
+Text GLabel 10725 3475 2    50   Input ~ 0
 A9
-Text GLabel 10750 2400 2    50   Input ~ 0
+Text GLabel 10725 3375 2    50   Input ~ 0
 A10
-Text GLabel 10750 2300 2    50   Input ~ 0
+Text GLabel 10725 3275 2    50   Input ~ 0
 A11
-Text GLabel 10750 2200 2    50   Input ~ 0
+Text GLabel 10725 3175 2    50   Input ~ 0
 A12
-Text GLabel 10750 2100 2    50   Input ~ 0
+Text GLabel 10725 3075 2    50   Input ~ 0
 A13
-Text GLabel 10750 2000 2    50   Input ~ 0
+Text GLabel 10725 2975 2    50   Input ~ 0
 A14
-Text GLabel 10750 1900 2    50   Input ~ 0
+Text GLabel 10725 2875 2    50   Input ~ 0
 A15
-Text GLabel 10750 1800 2    50   Input ~ 0
+Text GLabel 10725 2775 2    50   Input ~ 0
 A3
-Text GLabel 10750 1700 2    50   Input ~ 0
+Text GLabel 10725 2675 2    50   Input ~ 0
 A2
-Text GLabel 10750 1600 2    50   Input ~ 0
+Text GLabel 10725 2575 2    50   Input ~ 0
 A1
-Text GLabel 10750 1500 2    50   Input ~ 0
+Text GLabel 10725 2475 2    50   Input ~ 0
 A0
-Text GLabel 9850 2500 0    50   Input ~ 0
+Text GLabel 9825 3475 0    50   Input ~ 0
 WR
-Text GLabel 9850 2400 0    50   Input ~ 0
+Text GLabel 9825 3375 0    50   Input ~ 0
 RD
-Text GLabel 9850 2300 0    50   Input ~ 0
+Text GLabel 9825 3275 0    50   Input ~ 0
 IORQ
-Text GLabel 9850 2200 0    50   Input ~ 0
+Text GLabel 9825 3175 0    50   Input ~ 0
 MREQ
-Text GLabel 9850 2100 0    50   Input ~ 0
+Text GLabel 9825 3075 0    50   Input ~ 0
 HALT
-Text GLabel 9850 2000 0    50   Input ~ 0
+Text GLabel 9825 2975 0    50   Input ~ 0
 NMI
-Text GLabel 9850 1900 0    50   Input ~ 0
+Text GLabel 9825 2875 0    50   Input ~ 0
 INT
-Text GLabel 9850 1800 0    50   Input ~ 0
+Text GLabel 9825 2775 0    50   Input ~ 0
 D4'
-Text GLabel 9850 1700 0    50   Input ~ 0
+Text GLabel 9825 2675 0    50   Input ~ 0
 D3'
-Text GLabel 9850 1600 0    50   Input ~ 0
+Text GLabel 9825 2575 0    50   Input ~ 0
 D5'
-Text GLabel 9850 1500 0    50   Input ~ 0
+Text GLabel 9825 2475 0    50   Input ~ 0
 D6'
-Text GLabel 9850 1400 0    50   Input ~ 0
+Text GLabel 9825 2375 0    50   Input ~ 0
 D2'
-Text GLabel 9850 1300 0    50   Input ~ 0
+Text GLabel 9825 2275 0    50   Input ~ 0
 D1'
-Text GLabel 9850 1200 0    50   Input ~ 0
+Text GLabel 9825 2175 0    50   Input ~ 0
 D0'
-Text GLabel 9850 1000 0    50   Input ~ 0
+Text GLabel 9825 1975 0    50   Input ~ 0
 RAM_CS
-Text GLabel 9850 900  0    50   Input ~ 0
+Text GLabel 9825 1875 0    50   Input ~ 0
 D7'
 $Comp
 L power:GND #PWR0114
 U 1 1 5FDC26C4
-P 10750 1300
-F 0 "#PWR0114" H 10750 1050 50  0001 C CNN
-F 1 "GND" V 10750 1100 50  0000 C CNN
-F 2 "" H 10750 1300 50  0001 C CNN
-F 3 "" H 10750 1300 50  0001 C CNN
-	1    10750 1300
+P 10725 2275
+F 0 "#PWR0114" H 10725 2025 50  0001 C CNN
+F 1 "GND" V 10725 2075 50  0000 C CNN
+F 2 "" H 10725 2275 50  0001 C CNN
+F 3 "" H 10725 2275 50  0001 C CNN
+	1    10725 2275
 	0    -1   -1   0
 $EndComp
@@
 L power:GND #PWR0115
 U 1 1 5FDC1AD8
-P 10750 1200
-F 0 "#PWR0115" H 10750 950 50  0001 C CNN
-F 1 "GND" V 10750 1000 50  0000 C CNN
-F 2 "" H 10750 1200 50  0001 C CNN
-F 3 "" H 10750 1200 50  0001 C CNN
-	1    10750 1200
+P 10725 2175
+F 0 "#PWR0115" H 10725 1925 50  0001 C CNN
+F 1 "GND" V 10725 1975 50  0000 C CNN
+F 2 "" H 10725 2175 50  0001 C CNN
+F 3 "" H 10725 2175 50  0001 C CNN
+	1    10725 2175
 	0    -1   -1   0
 $EndComp
@@
 L power:+9V #PWR0116
 U 1 1 5FDC0646
-P 10750 1000
-F 0 "#PWR0116" H 10750 850 50  0001 C CNN
-F 1 "+9V" V 10750 1200 50  0000 C CNN
-F 2 "" H 10750 1000 50  0001 C CNN
-F 3 "" H 10750 1000 50  0001 C CNN
-	1    10750 1000
+P 10725 1975
+F 0 "#PWR0116" H 10725 1825 50  0001 C CNN
+F 1 "+9V" V 10725 2175 50  0000 C CNN
+F 2 "" H 10725 1975 50  0001 C CNN
+F 3 "" H 10725 1975 50  0001 C CNN
+	1    10725 1975
 	0    1    1    0
 $EndComp
@@
 L power:+5V #PWR0117
 U 1 1 5FDBF709
-P 10750 900
-F 0 "#PWR0117" H 10750 750 50  0001 C CNN
-F 1 "+5V" V 10750 1100 50  0000 C CNN
-F 2 "" H 10750 900 50  0001 C CNN
-F 3 "" H 10750 900 50  0001 C CNN
-	1    10750 900
+P 10725 1875
+F 0 "#PWR0117" H 10725 1725 50  0001 C CNN
+F 1 "+5V" V 10725 2075 50  0000 C CNN
+F 2 "" H 10725 1875 50  0001 C CNN
+F 3 "" H 10725 1875 50  0001 C CNN
+	1    10725 1875
 	0    1    1    0
 $EndComp
@@
 L Sinclair:ZX81BUS EDGE1
 U 1 1 5FD7DF00
-P 10300 1950
-F 0 "EDGE1" H 10300 3175 39  0000 C CNN
-F 1 "ZX81BUS" H 10300 3166 39  0001 C CNN
-F 2 "zxbus:ZX_Bus_Edge_Connector" H 10050 0   39  0001 C CNN
-F 3 "" H 10050 0   39  0001 C CNN
-	1    10300 1950
+P 10275 2925
+F 0 "EDGE1" H 10275 4150 39  0000 C CNN
+F 1 "ZX81BUS" H 10275 4141 39  0001 C CNN
+F 2 "zxbus:ZX_Bus_Edge_Connector" H 10025 975 39  0001 C CNN
+F 3 "" H 10025 975 39  0001 C CNN
+	1    10275 2925
 	1    0    0    -1
 $EndComp
@@
 Wire Wire Line
 	4375 1550 4375 1125
-Text GLabel 10750 1400 2    50   Input ~ 0
+Text GLabel 10725 2375 2    50   Input ~ 0
 CLK
 Wire Wire Line
@@
 ROW8
 $Sheet
-S 9650 3525 1100 325
+S 9725 6025 1100 325
 U 632617C4
 F0 "Extras" 50
@@
 P 8275 1025
 F 0 "IC102" V 8250 875 50  0000 L CNN
-F 1 "74HCT00" V 8450 625 50  0000 L CNN
+F 1 "74HCT00" V 8500 650 50  0000 L CNN
 F 2 "Housings_SOIC:SOIC-14_3.9x8.7mm_Pitch1.27mm" H 8275 1025 50  0001 C CNN
 F 3 "http://www.ti.com/lit/gpn/sn74hct00" H 8275 1025 50  0001 C CNN
@@
 L Connector:Conn_01x02 J2
 U 1 1 5FEF73ED
-P 8800 675
-F 0 "J2" H 8880 667 50  0000 L CNN
-F 1 "Conn_01x02" H 8880 576 50  0001 L CNN
-F 2 "Pin_Headers:Pin_Header_Straight_1x02_Pitch2.54mm" H 8800 675 50  0001 C CNN
-F 3 "~" H 8800 675 50  0001 C CNN
-	1    8800 675
+P 8950 675
+F 0 "J2" H 9030 667 50  0000 L CNN
+F 1 "Conn_01x02" H 9030 576 50  0001 L CNN
+F 2 "Pin_Headers:Pin_Header_Straight_1x02_Pitch2.54mm" H 8950 675 50  0001 C CNN
+F 3 "~" H 8950 675 50  0001 C CNN
+	1    8950 675
 	1    0    0    -1
 $EndComp
@@
 L power:GND #PWR0154
 U 1 1 5FF29BAB
-P 9175 900
-F 0 "#PWR0154" H 9175 650 50  0001 C CNN
-F 1 "GND" V 9275 925 50  0000 R CNN
-F 2 "" H 9175 900 50  0001 C CNN
-F 3 "" H 9175 900 50  0001 C CNN
-	1    9175 900
+P 9800 1575
+F 0 "#PWR0154" H 9800 1325 50  0001 C CNN
+F 1 "GND" V 9900 1600 50  0000 R CNN
+F 2 "" H 9800 1575 50  0001 C CNN
+F 3 "" H 9800 1575 50  0001 C CNN
+	1    9800 1575
 	1    0    0    -1
 $EndComp
@@
 L power:+5V #PWR0155
 U 1 1 5FF3B39F
-P 9275 575
-F 0 "#PWR0155" H 9275 425 50  0001 C CNN
-F 1 "+5V" V 9225 625 50  0000 L CNN
-F 2 "" H 9275 575 50  0001 C CNN
-F 3 "" H 9275 575 50  0001 C CNN
-	1    9275 575
+P 9875 575
+F 0 "#PWR0155" H 9875 425 50  0001 C CNN
+F 1 "+5V" V 9825 625 50  0000 L CNN
+F 2 "" H 9875 575 50  0001 C CNN
+F 3 "" H 9875 575 50  0001 C CNN
+	1    9875 575
 	0    1    1    0
 $EndComp
@@
 L device:C C105
 U 1 1 6000A744
-P 9175 750
-F 0 "C105" H 9290 796 50  0000 L CNN
-F 1 "100N" H 9290 705 50  0000 L CNN
-F 2 "Capacitors_SMD:C_0603_HandSoldering" H 9213 600 50  0001 C CNN
-F 3 "" H 9175 750 50  0001 C CNN
-	1    9175 750
+P 9275 900
+F 0 "C105" H 9075 1000 50  0000 L CNN
+F 1 "100N" H 9075 800 50  0000 L CNN
+F 2 "Capacitors_SMD:C_0603_HandSoldering" H 9313 750 50  0001 C CNN
+F 3 "" H 9275 900 50  0001 C CNN
+	1    9275 900
 	1    0    0    -1
 $EndComp
@@
 Wire Wire Line
 	25675 -12450 25675 -13400
-Wire Wire Line
-	8675 575  9175 575
-Wire Wire Line
-	9175 575  9175 600
-Connection ~ 9175 575
-Wire Wire Line
-	9175 575  9275 575
-Wire Wire Line
-	9175 900  8600 900
-Wire Wire Line
-	8600 900  8600 775
-Connection ~ 9175 900
-Wire Wire Line
-	8600 675  8375 675
 Connection ~ 8375 675
 Wire Wire Line
@@
 	-1   0    0    1
 $EndComp
+$Comp
+L Logic_74xx:74HCT00 IC102
+U 5 1 5FC8AE73
+P 9800 1075
+F 0 "IC102" H 10030 1121 50  0000 L CNN
+F 1 "74HCT00" H 10030 1030 50  0000 L CNN
+F 2 "" H 9800 1075 50  0001 C CNN
+F 3 "http://www.ti.com/lit/gpn/sn74hct00" H 9800 1075 50  0001 C CNN
+	5    9800 1075
+	1    0    0    -1
+$EndComp
+Wire Wire Line
+	9800 1575 9550 1575
+Wire Wire Line
+	9550 1575 9550 1275
+Connection ~ 9800 1575
+Wire Wire Line
+	9875 575  9800 575
+Connection ~ 9800 575
+Wire Wire Line
+	9550 1275 9275 1275
+Wire Wire Line
+	9275 1050 9275 1275
+Connection ~ 9275 1275
+Wire Wire Line
+	9275 1275 8750 1275
+Wire Wire Line
+	9275 750  9275 575
+Connection ~ 9275 575
+Wire Wire Line
+	9275 575  9800 575
+Wire Wire Line
+	8375 675  8750 675
+Wire Wire Line
+	8750 775  8750 1275
+Wire Wire Line
+	8675 575  9275 575
 $EndSCHEMATC

Commit message: 3 SD working better
Parts:
- IC1, IC3: footprint Housings_DIP:DIP-40_W15.24mm_Socket_LongPads -> zxbus:DIP-40_W15.24mm_Socket_LongPads
- IC102: footprint (none) -> Housings_SOIC:SOIC-14_3.9x8.7mm_Pitch1.27mm
- IC2, IC4: footprint Housings_DIP:DIP-28_W15.24mm_Socket_LongPads -> zxbus:DIP-28_W15.24mm_Socket_LongPads
Changed lines of the file:
@@
 F 0 "IC2" H 5200 5225 50  0000 C CNN
 F 1 "AT28C256" H 5200 5125 50  0000 C CNN
-F 2 "Housings_DIP:DIP-28_W15.24mm_Socket_LongPads" H 5200 5025 50  0001 C CNN
+F 2 "zxbus:DIP-28_W15.24mm_Socket_LongPads" H 5200 5025 50  0001 C CNN
 F 3 "" H 5200 5025 50  0001 C CNN
 	1    5200 5325
@@
 F 0 "IC1" H 2750 3325 50  0000 C CNN
 F 1 "ULA 2C210E" H 2750 3175 50  0000 C CNN
-F 2 "Housings_DIP:DIP-40_W15.24mm_Socket_LongPads" H 3450 3725 50  0001 C CNN
+F 2 "zxbus:DIP-40_W15.24mm_Socket_LongPads" H 3450 3725 50  0001 C CNN
 F 3 "" H 3450 3725 50  0001 C CNN
 	1    2750 3025
@@
 F 0 "IC4" V 7600 3675 50  0000 C CNN
 F 1 "62256" V 7700 3675 50  0000 C CNN
-F 2 "Housings_DIP:DIP-28_W15.24mm_Socket_LongPads" H 7650 3625 50  0001 C CIN
+F 2 "zxbus:DIP-28_W15.24mm_Socket_LongPads" H 7650 3625 50  0001 C CIN
 F 3 "" H 7650 3625 50  0001 C CNN
 	1    7650 3625
@@
 F 0 "IC3" H 5450 2725 50  0000 C CNN
 F 1 "Z80A" H 5450 2625 50  0000 C CNN
-F 2 "Housings_DIP:DIP-40_W15.24mm_Socket_LongPads" H 5450 3025 50  0001 C CNN
+F 2 "zxbus:DIP-40_W15.24mm_Socket_LongPads" H 5450 3025 50  0001 C CNN
 F 3 "www.zilog.com/manage_directlink.php?filepath=docs/z80/um0080" H 5450 3025 50  0001 C CNN
 	1    5450 2625
@@
 F 0 "IC102" H 10030 1121 50  0000 L CNN
 F 1 "74HCT00" H 10030 1030 50  0000 L CNN
-F 2 "" H 9800 1075 50  0001 C CNN
+F 2 "Housings_SOIC:SOIC-14_3.9x8.7mm_Pitch1.27mm" H 9800 1075 50  0001 C CNN
 F 3 "http://www.ti.com/lit/gpn/sn74hct00" H 9800 1075 50  0001 C CNN
 	5    9800 1075

Commit message: Yup more routing
Parts:
- removed J2: Conn_01x02, Pin_Headers:Pin_Header_Straight_1x02_Pitch2.54mm, symbol Connector:Conn_01x02
- added J101: Conn_01x03, Pin_Headers:Pin_Header_Straight_1x03_Pitch2.54mm, symbol Connector:Conn_01x03
- added R106: 10K, Resistors_SMD:R_0603_HandSoldering, symbol device:R
- R105: value 4K7 -> 10K
Connections:
- wire segments 439 -> 444
Other:
- moved on the sheet: IC102A, IC102B, IC102C, IC102D, R105
Changed lines of the file:
@@
 L Logic_74xx:74HCT00 IC102
 U 1 1 5FD1E154
-P 7100 1025
-F 0 "IC102" V 7075 900 50  0000 L CNN
-F 1 "74HCT00" V 7375 2525 50  0001 L CNN
-F 2 "Housings_SOIC:SOIC-14_3.9x8.7mm_Pitch1.27mm" H 7100 1025 50  0001 C CNN
-F 3 "http://www.ti.com/lit/gpn/sn74hct00" H 7100 1025 50  0001 C CNN
-	1    7100 1025
+P 7100 1075
+F 0 "IC102" V 7075 950 50  0000 L CNN
+F 1 "74HCT00" V 7375 2575 50  0001 L CNN
+F 2 "Housings_SOIC:SOIC-14_3.9x8.7mm_Pitch1.27mm" H 7100 1075 50  0001 C CNN
+F 3 "http://www.ti.com/lit/gpn/sn74hct00" H 7100 1075 50  0001 C CNN
+	1    7100 1075
 	0    1    1    0
 $EndComp
@@
 L Logic_74xx:74HCT00 IC102
 U 2 1 5FD21B16
-P 7500 1025
-F 0 "IC102" V 7475 875 50  0000 L CNN
-F 1 "74HCT00" H 7600 1175 50  0001 L CNN
-F 2 "Housings_SOIC:SOIC-14_3.9x8.7mm_Pitch1.27mm" H 7500 1025 50  0001 C CNN
-F 3 "http://www.ti.com/lit/gpn/sn74hct00" H 7500 1025 50  0001 C CNN
-	2    7500 1025
+P 7500 1075
+F 0 "IC102" V 7475 925 50  0000 L CNN
+F 1 "74HCT00" H 7600 1225 50  0001 L CNN
+F 2 "Housings_SOIC:SOIC-14_3.9x8.7mm_Pitch1.27mm" H 7500 1075 50  0001 C CNN
+F 3 "http://www.ti.com/lit/gpn/sn74hct00" H 7500 1075 50  0001 C CNN
+	2    7500 1075
 	0    1    1    0
 $EndComp
@@
 L Logic_74xx:74HCT00 IC102
 U 3 1 5FD24E41
-P 7900 1025
-F 0 "IC102" V 7875 900 50  0000 L CNN
-F 1 "74HCT00" V 7945 1213 50  0001 L CNN
-F 2 "Housings_SOIC:SOIC-14_3.9x8.7mm_Pitch1.27mm" H 7900 1025 50  0001 C CNN
-F 3 "http://www.ti.com/lit/gpn/sn74hct00" H 7900 1025 50  0001 C CNN
-	3    7900 1025
+P 7900 1075
+F 0 "IC102" V 7875 950 50  0000 L CNN
+F 1 "74HCT00" V 7945 1263 50  0001 L CNN
+F 2 "Housings_SOIC:SOIC-14_3.9x8.7mm_Pitch1.27mm" H 7900 1075 50  0001 C CNN
+F 3 "http://www.ti.com/lit/gpn/sn74hct00" H 7900 1075 50  0001 C CNN
+	3    7900 1075
 	0    -1   1    0
 $EndComp
@@
 L Logic_74xx:74HCT00 IC102
 U 4 1 5FD25FC1
-P 8275 1025
-F 0 "IC102" V 8250 875 50  0000 L CNN
-F 1 "74HCT00" V 8500 650 50  0000 L CNN
-F 2 "Housings_SOIC:SOIC-14_3.9x8.7mm_Pitch1.27mm" H 8275 1025 50  0001 C CNN
-F 3 "http://www.ti.com/lit/gpn/sn74hct00" H 8275 1025 50  0001 C CNN
-	4    8275 1025
+P 8275 1075
+F 0 "IC102" V 8250 925 50  0000 L CNN
+F 1 "74HCT00" V 8500 700 50  0000 L CNN
+F 2 "Housings_SOIC:SOIC-14_3.9x8.7mm_Pitch1.27mm" H 8275 1075 50  0001 C CNN
+F 3 "http://www.ti.com/lit/gpn/sn74hct00" H 8275 1075 50  0001 C CNN
+	4    8275 1075
 	0    -1   1    0
 $EndComp
 Wire Wire Line
-	7100 3125 7100 1325
-Wire Wire Line
-	7200 3125 7200 1325
-Wire Wire Line
-	7200 1325 7500 1325
-Wire Wire Line
-	7300 3125 7300 1375
-Wire Wire Line
-	7300 1375 7900 1375
-Wire Wire Line
-	7900 1375 7900 1325
-Wire Wire Line
-	8275 1325 8275 1450
-Wire Wire Line
-	8275 1450 7400 1450
-Wire Wire Line
-	7400 1450 7400 3125
-Text GLabel 7000 725  1    50   Input ~ 0
+	7200 3125 7200 1375
+Wire Wire Line
+	7200 1375 7500 1375
+Wire Wire Line
+	7300 3125 7300 1425
+Wire Wire Line
+	7300 1425 7900 1425
+Wire Wire Line
+	8275 1475 7400 1475
+Wire Wire Line
+	7400 1475 7400 3125
+Text GLabel 7000 775  1    50   Input ~ 0
 A13
-Text GLabel 7400 725  1    50   Input ~ 0
+Text GLabel 7400 775  1    50   Input ~ 0
 A12
-Text GLabel 7800 725  1    50   Input ~ 0
+Text GLabel 7800 775  1    50   Input ~ 0
 A11
-Text GLabel 8175 725  1    50   Input ~ 0
+Text GLabel 8175 775  1    50   Input ~ 0
 A10
-Wire Wire Line
-	7200 725  7200 500
-Wire Wire Line
-	7200 500  7600 500
-Wire Wire Line
-	8375 500  8375 575
-Wire Wire Line
-	8000 725  8000 500
-Connection ~ 8000 500
-Wire Wire Line
-	8000 500  8375 500
-Wire Wire Line
-	7600 725  7600 500
-Connection ~ 7600 500
-Wire Wire Line
-	7600 500  8000 500
-$Comp
-L Connector:Conn_01x02 J2
-U 1 1 5FEF73ED
-P 8950 675
-F 0 "J2" H 9030 667 50  0000 L CNN
-F 1 "Conn_01x02" H 9030 576 50  0001 L CNN
-F 2 "Pin_Headers:Pin_Header_Straight_1x02_Pitch2.54mm" H 8950 675 50  0001 C CNN
-F 3 "~" H 8950 675 50  0001 C CNN
-	1    8950 675
-	1    0    0    -1
-$EndComp
 $Comp
 L power:GND #PWR0154
@@
 L device:R R105
 U 1 1 5FF3AB29
-P 8525 575
-F 0 "R105" V 8525 575 50  0000 C CNN
-F 1 "4K7" V 8575 375 50  0000 C CNN
-F 2 "Resistors_SMD:R_0603_HandSoldering" V 8455 575 50  0001 C CNN
-F 3 "" H 8525 575 50  0001 C CNN
-	1    8525 575
+P 8925 575
+F 0 "R105" V 8925 575 50  0000 C CNN
+F 1 "10K" V 8975 375 50  0000 C CNN
+F 2 "Resistors_SMD:R_0603_HandSoldering" V 8855 575 50  0001 C CNN
+F 3 "" H 8925 575 50  0001 C CNN
+	1    8925 575
 	0    -1   -1   0
 $EndComp
-Connection ~ 8375 575
 $Comp
 L power:+5V #PWR0155
@@
 	0    1    1    0
 $EndComp
-Wire Wire Line
-	8375 575  8375 675
 $Comp
 L device:C C105
@@
 Wire Wire Line
 	25675 -12450 25675 -13400
-Connection ~ 8375 675
-Wire Wire Line
-	8375 675  8375 725
 Wire Wire Line
 	3650 4625 8400 4625
@@
 Wire Wire Line
 	9275 1050 9275 1275
+Wire Wire Line
+	9275 575  9800 575
+$Comp
+L device:R R106
+U 1 1 5FC6BFB3
+P 8925 725
+F 0 "R106" V 8925 725 50  0000 C CNN
+F 1 "10K" V 8975 525 50  0000 C CNN
+F 2 "Resistors_SMD:R_0603_HandSoldering" V 8855 725 50  0001 C CNN
+F 3 "" H 8925 725 50  0001 C CNN
+	1    8925 725
+	0    -1   -1   0
+$EndComp
+$Comp
+L Connector:Conn_01x03 J101
+U 1 1 5FC6F451
+P 8750 1175
+F 0 "J101" V 8850 1150 50  0000 L CNN
+F 1 "Conn_01x03" H 8830 1126 50  0001 L CNN
+F 2 "Pin_Headers:Pin_Header_Straight_1x03_Pitch2.54mm" H 8750 1175 50  0001 C CNN
+F 3 "~" H 8750 1175 50  0001 C CNN
+	1    8750 1175
+	0    1    1    0
+$EndComp
+Wire Wire Line
+	9275 575  9075 575
+Connection ~ 9275 575
+Wire Wire Line
+	8775 575  8650 575
+Connection ~ 8000 575
+Wire Wire Line
+	8650 975  8650 575
+Connection ~ 8650 575
+Wire Wire Line
+	8650 575  8000 575
+Wire Wire Line
+	9275 575  9275 725
+Wire Wire Line
+	8750 975  8750 725
+Wire Wire Line
+	8775 725  8750 725
+Wire Wire Line
+	9075 725  9275 725
+Connection ~ 9275 725
+Wire Wire Line
+	9275 725  9275 750
+Wire Wire Line
+	9275 1275 9025 1275
+Wire Wire Line
+	9025 1275 9025 975
+Wire Wire Line
+	9025 975  8850 975
 Connection ~ 9275 1275
 Wire Wire Line
-	9275 1275 8750 1275
-Wire Wire Line
-	9275 750  9275 575
-Connection ~ 9275 575
-Wire Wire Line
-	9275 575  9800 575
-Wire Wire Line
-	8375 675  8750 675
-Wire Wire Line
-	8750 775  8750 1275
-Wire Wire Line
-	8675 575  9275 575
+	7200 575  7200 775
+Wire Wire Line
+	8000 575  8000 775
+Wire Wire Line
+	7600 575  7600 775
+Wire Wire Line
+	7900 1425 7900 1375
+Wire Wire Line
+	8275 1475 8275 1375
+Wire Wire Line
+	7100 3125 7100 1375
+Wire Wire Line
+	7200 575  7600 575
+Connection ~ 7600 575
+Wire Wire Line
+	7600 575  8000 575
+Wire Wire Line
+	8750 725  8375 725
+Wire Wire Line
+	8375 725  8375 775
+Connection ~ 8750 725
 $EndSCHEMATC

Commit message: Fixing DRC Issues
Parts:
- C1: footprint Capacitors_THT:C_Disc_D4.7mm_W2.5mm_P5.00mm -> Capacitors_THT:C_Disc_D3.0mm_W2.0mm_P2.50mm
- C10, C102, C103, C104, C11, C12, C4, C6, C7, C8, C9: footprint Capacitors_THT:C_Disc_D4.7mm_W2.5mm_P5.00mm -> Capacitors_ThroughHole:C_Disc_D4.7mm_W2.5mm_P5.00mm
- C3: footprint Capacitors_THT:CP_Axial_L11.0mm_D5.0mm_P18.00mm_Horizontal -> Capacitors_ThroughHole:CP_Axial_L11.0mm_D5.0mm_P18.00mm_Horizontal
- C5: footprint Capacitors_THT:CP_Radial_D5.0mm_P2.50mm -> Capacitors_ThroughHole:CP_Radial_D5.0mm_P2.50mm
- D1, D101, D102, D2, D3, D4, D5, D6, D7, D8: footprint Diodes_THT:D_DO-35_SOD27_P7.62mm_Horizontal -> zxbus:D_DO-35_SOD27_P7.62mm_Horizontal
- R1, R10, R101, R102, R103, R104, R11, R12, R13, R14, R15, R16, R17, R18, R19, R2, R20, R201, R21, R22, R23, R24, R25, R26, R27, R28, R29, R30, R33, R34, R4, R5, R6, R7, R8, R9: footprint Resistors_ThroughHole:R_Axial_DIN0207_L6.3mm_D2.5mm_P7.62mm_Horizontal -> Resistors_ThroughHole:R_Axial_DIN0204_L3.6mm_D1.6mm_P7.62mm_Horizontal

Commit message: FIrst go at DRC complete
Parts:
- J101, J203, J204: footprint Pin_Headers:Pin_Header_Straight_1x03_Pitch2.54mm -> zxbus:Pin_Header_Straight_1x03_Pitch2.54mm
- S1: footprint SamacSys_Parts:EG4208A -> SamacSys_Parts:EG4208
Changed lines of the file:
@@
 F 0 "J204" V 4125 6925 50  0000 L CNN
 F 1 "Conn_01x03" H 4205 7226 50  0001 L CNN
-F 2 "Pin_Headers:Pin_Header_Straight_1x03_Pitch2.54mm" H 4125 7275 50  0001 C CNN
+F 2 "zxbus:Pin_Header_Straight_1x03_Pitch2.54mm" H 4125 7275 50  0001 C CNN
 F 3 "~" H 4125 7275 50  0001 C CNN
 	1    4125 7275
@@
 F 0 "J203" V 4500 7450 50  0000 L CNN
 F 1 "Conn_01x03" H 4580 7226 50  0001 L CNN
-F 2 "Pin_Headers:Pin_Header_Straight_1x03_Pitch2.54mm" H 4500 7275 50  0001 C CNN
+F 2 "zxbus:Pin_Header_Straight_1x03_Pitch2.54mm" H 4500 7275 50  0001 C CNN
 F 3 "~" H 4500 7275 50  0001 C CNN
 	1    4500 7275
@@
 F 0 "S1" H 5525 7450 50  0000 C CNN
 F 1 "EG4208A" H 5925 7450 50  0000 C CNN
-F 2 "SamacSys_Parts:EG4208A" H 6300 7450 50  0001 L CNN
+F 2 "SamacSys_Parts:EG4208" H 6300 7450 50  0001 L CNN
 F 3 "https://www.e-switch.com/system/asset/product_line/data_sheet/119/EG.pdf" H 4600 7750 50  0001 L CNN
 F 4 "Slide Switches 4P2T SIDE OP PC MNT" H 4600 7850 50  0001 L CNN "Description"
@@
 F 0 "J101" V 8850 1150 50  0000 L CNN
 F 1 "Conn_01x03" H 8830 1126 50  0001 L CNN
-F 2 "Pin_Headers:Pin_Header_Straight_1x03_Pitch2.54mm" H 8750 1175 50  0001 C CNN
+F 2 "zxbus:Pin_Header_Straight_1x03_Pitch2.54mm" H 8750 1175 50  0001 C CNN
 F 3 "~" H 8750 1175 50  0001 C CNN
 	1    8750 1175

Commit message: ESP32 Flipped
Parts:
- C101: footprint Capacitors_ThroughHole:CP_Axial_L11.0mm_D5.0mm_P18.00mm_Horizontal -> Capacitors_ThroughHole:CP_Radial_D5.0mm_P2.50mm
Changed lines of the file:
@@
 F 0 "C101" H 2050 1375 50  0000 L CNN
 F 1 "22U" H 2125 1275 50  0000 L CNN
-F 2 "Capacitors_ThroughHole:CP_Axial_L11.0mm_D5.0mm_P18.00mm_Horizontal" H 2163 1025 50  0001 C CNN
+F 2 "Capacitors_ThroughHole:CP_Radial_D5.0mm_P2.50mm" H 2163 1025 50  0001 C CNN
 F 3 "" H 2125 1175 50  0001 C CNN
 	1    2125 1175
