File: KiCad/ZX21/ZX21_Extras.sch (KiCad schematic (older format))
At the start: 17 parts, among them IC301 3V3 PSU, IC302 ESP32-WROOM, IC303 AZ1117-3.3, IC501 YM2149, J401 DB9_Male

Commit message: Extras first draft
Parts:
- added J501: Conn_01x05, symbol Connector:Conn_01x05
- added J502, J503: Conn_01x08, symbol Connector:Conn_01x08
- added J504: Conn_01x07, symbol Connector:Conn_01x07
- added J601: Conn_02x08_Odd_Even, symbol Connector:Conn_02x08_Odd_Even
- added J701: Conn_02x23_Row_Letter_First, symbol Connector:Conn_02x23_Row_Letter_First
- added J702: Conn_01x09, symbol Connector:Conn_01x09
- added R501, R502, R503: 4K7, symbol device:R
- added R504: 1K, symbol device:R
- added UIC502: GAL16V8, symbol Lattice:GAL16V8
- gave numbers to parts that had none: 1
Connections:
- net labels added: A0, A1, A10, A11, A12, A13, A14, A15, A2, A3, A4, A5, A6, A7, A8, A9, BUSAK, BUSRQ, CLK, D0, D1, D2, D3, D4, D5, D6, D7, HALT, INT, IORQ, KBD1, KBD5, MI, MREQ, NMI, RAM_CS, RD, RESET, RFSH, ROM_CS, ROW2, ROW3, ROW5, ROW6, ROW7, ROW8, SOUND, WAIT, WR
- wire segments 60 -> 88
- no-connect marks 6 -> 7
Other:
- note added: "dK'tronics\nKEYBOARD"
- moved on the sheet: IC501, J401, QTR403, R401, TR401, TR402, TR404, TR405

Commit message: Fixed most ERC Issues
Parts:
- added J703: Conn_01x09, symbol Connector:Conn_01x09
Connections:
- net labels added: A0', A1', A2', A3', A4', A5', A6', A7', A8'
- net labels removed: KBD5
- no-connect marks 7 -> 39
Other:
- moved on the sheet: J702
Changed lines of the file:
@@
 $EndComp
 $Comp
-L power:GND #PWR?
+L power:GND #PWR0131
 U 1 1 63266B61
 P 2100 3225
-F 0 "#PWR?" H 2100 2975 50  0001 C CNN
+F 0 "#PWR0131" H 2100 2975 50  0001 C CNN
 F 1 "GND" H 2105 3052 50  0000 C CNN
 F 2 "" H 2100 3225 50  0001 C CNN
@@
 	1475 1500 1550 1500
 $Comp
-L power:+9V #PWR?
+L power:+9V #PWR0132
 U 1 1 6326A474
 P 800 1500
-F 0 "#PWR?" H 800 1350 50  0001 C CNN
+F 0 "#PWR0132" H 800 1350 50  0001 C CNN
 F 1 "+9V" H 815 1673 50  0000 C CNN
 F 2 "" H 800 1500 50  0001 C CNN
@@
 Connection ~ 875  1500
 $Comp
-L power:GND #PWR?
+L power:GND #PWR0133
 U 1 1 6327B84A
 P 1175 1150
-F 0 "#PWR?" H 1175 900 50  0001 C CNN
+F 0 "#PWR0133" H 1175 900 50  0001 C CNN
 F 1 "GND" V 1180 1022 50  0000 R CNN
 F 2 "" H 1175 1150 50  0001 C CNN
@@
 $EndComp
 $Comp
-L power:+5V #PWR?
+L power:+5V #PWR0134
 U 1 1 63340297
 P 9500 1475
-F 0 "#PWR?" H 9500 1325 50  0001 C CNN
+F 0 "#PWR0134" H 9500 1325 50  0001 C CNN
 F 1 "+5V" H 9515 1648 50  0000 C CNN
 F 2 "" H 9500 1475 50  0001 C CNN
@@
 D7'
 $Comp
-L power:+5V #PWR?
+L power:+5V #PWR0135
 U 1 1 6337138B
 P 9400 3325
-F 0 "#PWR?" H 9400 3175 50  0001 C CNN
+F 0 "#PWR0135" H 9400 3175 50  0001 C CNN
 F 1 "+5V" H 9415 3498 50  0000 C CNN
 F 2 "" H 9400 3325 50  0001 C CNN
@@
 NoConn ~ 9700 3325
 $Comp
-L power:GND #PWR?
+L power:GND #PWR0136
 U 1 1 63374D25
 P 9400 6125
-F 0 "#PWR?" H 9400 5875 50  0001 C CNN
+F 0 "#PWR0136" H 9400 5875 50  0001 C CNN
 F 1 "GND" H 9405 5952 50  0000 C CNN
 F 2 "" H 9400 6125 50  0001 C CNN
@@
 $EndComp
 $Comp
-L power:GND #PWR?
+L power:GND #PWR0137
 U 1 1 63377A27
 P 1475 3700
-F 0 "#PWR?" H 1475 3450 50  0001 C CNN
+F 0 "#PWR0137" H 1475 3450 50  0001 C CNN
 F 1 "GND" V 1480 3572 50  0000 R CNN
 F 2 "" H 1475 3700 50  0001 C CNN
@@
 $EndComp
 $Comp
-L power:GND #PWR?
+L power:GND #PWR0138
 U 1 1 5FC9B6C5
 P 10575 4175
-F 0 "#PWR?" H 10575 3925 50  0001 C CNN
+F 0 "#PWR0138" H 10575 3925 50  0001 C CNN
 F 1 "GND" H 10580 4002 50  0000 C CNN
 F 2 "" H 10575 4175 50  0001 C CNN
@@
 	8375 4075 7450 4075
 $Comp
-L power:GND #PWR?
+L power:GND #PWR0139
 U 1 1 5FCD4A93
 P 7450 4175
-F 0 "#PWR?" H 7450 3925 50  0001 C CNN
+F 0 "#PWR0139" H 7450 3925 50  0001 C CNN
 F 1 "GND" V 7455 4047 50  0000 R CNN
 F 2 "" H 7450 4175 50  0001 C CNN
@@
 $EndComp
 $Comp
-L power:+5V #PWR?
+L power:+5V #PWR0140
 U 1 1 5FCD57A2
 P 7450 3575
-F 0 "#PWR?" H 7450 3425 50  0001 C CNN
+F 0 "#PWR0140" H 7450 3425 50  0001 C CNN
 F 1 "+5V" V 7465 3703 50  0000 L CNN
 F 2 "" H 7450 3575 50  0001 C CNN
@@
 Connection ~ 4175 2750
 $Comp
-L power:+5V #PWR?
+L power:+5V #PWR0141
 U 1 1 5FCD96A1
 P 1475 3400
-F 0 "#PWR?" H 1475 3250 50  0001 C CNN
+F 0 "#PWR0141" H 1475 3250 50  0001 C CNN
 F 1 "+5V" V 1490 3528 50  0000 L CNN
 F 2 "" H 1475 3400 50  0001 C CNN
@@
 ROW7
 $Comp
-L power:+5V #PWR?
+L power:+5V #PWR0142
 U 1 1 5FCF7BBB
 P 5725 1675
-F 0 "#PWR?" H 5725 1525 50  0001 C CNN
+F 0 "#PWR0142" H 5725 1525 50  0001 C CNN
 F 1 "+5V" V 5700 1800 50  0000 L CNN
 F 2 "" H 5725 1675 50  0001 C CNN
@@
 $EndComp
 $Comp
-L power:GND #PWR?
+L power:GND #PWR0143
 U 1 1 5FCF8527
 P 5725 1775
-F 0 "#PWR?" H 5725 1525 50  0001 C CNN
+F 0 "#PWR0143" H 5725 1525 50  0001 C CNN
 F 1 "GND" V 5725 1650 50  0000 R CNN
 F 2 "" H 5725 1775 50  0001 C CNN
@@
 ROW4
 Text GLabel 5725 2375 2    50   Input ~ 0
-KBD5
+KBD4
 Text GLabel 5225 2375 0    50   Input ~ 0
 ROW6
@@
 L Connector:Conn_01x09 J702
 U 1 1 5FD0553E
-P 8200 1975
-F 0 "J702" V 8300 1875 50  0000 L CNN
-F 1 "Conn_01x09" H 8280 1926 50  0001 L CNN
-F 2 "" H 8200 1975 50  0001 C CNN
-F 3 "~" H 8200 1975 50  0001 C CNN
-	1    8200 1975
+P 8350 2625
+F 0 "J702" V 8450 2525 50  0000 L CNN
+F 1 "Conn_01x09" H 8430 2576 50  0001 L CNN
+F 2 "" H 8350 2625 50  0001 C CNN
+F 3 "~" H 8350 2625 50  0001 C CNN
+	1    8350 2625
 	1    0    0    -1
 $EndComp
@@
 RFSH
 $Comp
-L power:GND #PWR?
+L power:GND #PWR0144
 U 1 1 5FD13F13
 P 6925 1075
-F 0 "#PWR?" H 6925 825 50  0001 C CNN
+F 0 "#PWR0144" H 6925 825 50  0001 C CNN
 F 1 "GND" V 6930 947 50  0000 R CNN
 F 2 "" H 6925 1075 50  0001 C CNN
@@
 $EndComp
 $Comp
-L power:GND #PWR?
+L power:GND #PWR0145
 U 1 1 5FD14A25
 P 7425 1075
-F 0 "#PWR?" H 7425 825 50  0001 C CNN
+F 0 "#PWR0145" H 7425 825 50  0001 C CNN
 F 1 "GND" V 7430 947 50  0000 R CNN
 F 2 "" H 7425 1075 50  0001 C CNN
@@
 $EndComp
 $Comp
-L power:GND #PWR?
+L power:GND #PWR0146
 U 1 1 5FD157B7
 P 7425 1175
-F 0 "#PWR?" H 7425 925 50  0001 C CNN
+F 0 "#PWR0146" H 7425 925 50  0001 C CNN
 F 1 "GND" V 7430 1047 50  0000 R CNN
 F 2 "" H 7425 1175 50  0001 C CNN
@@
 $EndComp
 $Comp
-L power:GND #PWR?
+L power:GND #PWR0147
 U 1 1 5FD161EE
 P 7425 1275
-F 0 "#PWR?" H 7425 1025 50  0001 C CNN
+F 0 "#PWR0147" H 7425 1025 50  0001 C CNN
 F 1 "GND" V 7430 1147 50  0000 R CNN
 F 2 "" H 7425 1275 50  0001 C CNN
@@
 $EndComp
 $Comp
-L power:+5V #PWR?
+L power:+5V #PWR0148
 U 1 1 5FD17049
 P 7425 875
-F 0 "#PWR?" H 7425 725 50  0001 C CNN
+F 0 "#PWR0148" H 7425 725 50  0001 C CNN
 F 1 "+5V" V 7440 1003 50  0000 L CNN
 F 2 "" H 7425 875 50  0001 C CNN
@@
 $EndComp
 $Comp
-L power:+9V #PWR?
+L power:+9V #PWR0149
 U 1 1 5FD175E6
 P 7425 975
-F 0 "#PWR?" H 7425 825 50  0001 C CNN
+F 0 "#PWR0149" H 7425 825 50  0001 C CNN
 F 1 "+9V" V 7440 1103 50  0000 L CNN
 F 2 "" H 7425 975 50  0001 C CNN
@@
 Text GLabel 7425 3075 2    50   Input ~ 0
 ROM_CS
-Text GLabel 8000 1675 0    50   Input ~ 0
+Text GLabel 8150 2325 0    50   Input ~ 0
 D0
-Text GLabel 8000 1775 0    50   Input ~ 0
+Text GLabel 8150 2425 0    50   Input ~ 0
 D1
-Text GLabel 8000 1875 0    50   Input ~ 0
+Text GLabel 8150 2525 0    50   Input ~ 0
 D2
-Text GLabel 8000 2075 0    50   Input ~ 0
+Text GLabel 8150 2725 0    50   Input ~ 0
 D4
 $Comp
-L power:GND #PWR?
+L power:GND #PWR0150
 U 1 1 5FD25F51
-P 8000 1575
-F 0 "#PWR?" H 8000 1325 50  0001 C CNN
-F 1 "GND" V 8005 1447 50  0000 R CNN
-F 2 "" H 8000 1575 50  0001 C CNN
-F 3 "" H 8000 1575 50  0001 C CNN
-	1    8000 1575
-	0    1    1    0
-$EndComp
-Text GLabel 8000 1975 0    50   Input ~ 0
+P 8150 2225
+F 0 "#PWR0150" H 8150 1975 50  0001 C CNN
+F 1 "GND" V 8155 2097 50  0000 R CNN
+F 2 "" H 8150 2225 50  0001 C CNN
+F 3 "" H 8150 2225 50  0001 C CNN
+	1    8150 2225
+	0    1    1    0
+$EndComp
+Text GLabel 8150 2625 0    50   Input ~ 0
 D3
-Text GLabel 8000 2175 0    50   Input ~ 0
+Text GLabel 8150 2825 0    50   Input ~ 0
 D5
-Text GLabel 8000 2275 0    50   Input ~ 0
+Text GLabel 8150 2925 0    50   Input ~ 0
 D6
-Text GLabel 8000 2375 0    50   Input ~ 0
+Text GLabel 8150 3025 0    50   Input ~ 0
 D7
+NoConn ~ 3950 1350
+NoConn ~ 3950 1550
+NoConn ~ 3950 1650
+NoConn ~ 3950 1750
+NoConn ~ 3950 1850
+NoConn ~ 3950 1950
+NoConn ~ 3950 2050
+NoConn ~ 3950 2150
+NoConn ~ 3950 2250
+NoConn ~ 3950 2350
+NoConn ~ 3950 2450
+NoConn ~ 3950 2550
+NoConn ~ 2100 2700
+NoConn ~ 2100 2600
+NoConn ~ 2100 2500
+NoConn ~ 2100 2400
+NoConn ~ 2100 2300
+NoConn ~ 2100 2200
+NoConn ~ 2100 2100
+NoConn ~ 2100 2000
+NoConn ~ 2100 1900
+NoConn ~ 2100 1800
+NoConn ~ 2700 3150
+NoConn ~ 2800 3150
+NoConn ~ 2900 3150
+NoConn ~ 3000 3150
+NoConn ~ 3100 3150
+NoConn ~ 3200 3150
+NoConn ~ 3300 3150
+NoConn ~ 3400 3150
+NoConn ~ 3500 3150
+$Comp
+L Connector:Conn_01x09 J703
+U 1 1 5FF5F4DB
+P 8350 1700
+F 0 "J703" V 8450 1575 50  0000 L CNN
+F 1 "Conn_01x09" H 8430 1651 50  0001 L CNN
+F 2 "" H 8350 1700 50  0001 C CNN
+F 3 "~" H 8350 1700 50  0001 C CNN
+	1    8350 1700
+	1    0    0    -1
+$EndComp
+Text GLabel 8150 1300 0    50   Input ~ 0
+A0'
+Text GLabel 8150 1400 0    50   Input ~ 0
+A1'
+Text GLabel 8150 1500 0    50   Input ~ 0
+A2'
+Text GLabel 8150 1600 0    50   Input ~ 0
+A3'
+Text GLabel 8150 1700 0    50   Input ~ 0
+A4'
+Text GLabel 8150 1800 0    50   Input ~ 0
+A5'
+Text GLabel 8150 1900 0    50   Input ~ 0
+A6'
+Text GLabel 8150 2000 0    50   Input ~ 0
+A7'
+Text GLabel 8150 2100 0    50   Input ~ 0
+A8'
+NoConn ~ 2100 1600
 $EndSCHEMATC

Commit message: Layout Started
Parts:
- C301, C302: footprint (none) -> Capacitors_THT:CP_Radial_D5.0mm_P2.50mm
- IC301: footprint (none) -> TO_SOT_Packages_THT:TO-220-3_Horizontal
- IC303: footprint (none) -> TO_SOT_Packages_SMD:SOT-23_Handsoldering
- IC501: footprint (none) -> Housings_DIP:DIP-40_W15.24mm_Socket_LongPads
- IC502: renamed from UIC502; footprint (none) -> Housings_DIP:DIP-20_W7.62mm_Socket_LongPads
- J301: footprint (none) -> Pin_Headers:Pin_Header_Straight_1x04_Pitch2.54mm
- J401: footprint (none) -> Connectors:DB9MC
- J501: footprint (none) -> Pin_Headers:Pin_Header_Straight_1x05_Pitch2.54mm
- J502, J503: footprint (none) -> Pin_Headers:Pin_Header_Straight_1x08_Pitch2.54mm
- J504: footprint (none) -> Pin_Headers:Pin_Header_Straight_1x07_Pitch2.54mm
- J601: footprint (none) -> Connectors:IDC_Header_Straight_16pins
- J701: footprint (none) -> Pin_Headers:Pin_Header_Straight_2x23_Pitch2.54mm
- J702, J703: footprint (none) -> Pin_Headers:Pin_Header_Straight_1x09_Pitch2.54mm
- R301, R302, R303, R401, R501, R502, R503, R504: footprint (none) -> Resistors_ThroughHole:R_Axial_DIN0207_L6.3mm_D2.5mm_P7.62mm_Horizontal
Changed lines of the file:
@@
 F 0 "IC301" H 1175 1742 50  0000 C CNN
 F 1 "3V3 PSU" H 1175 1651 50  0000 C CNN
-F 2 "" H 1200 1350 50  0001 L CIN
+F 2 "TO_SOT_Packages_THT:TO-220-3_Horizontal" H 1200 1350 50  0001 L CIN
 F 3 "http://www.st.com/content/ccc/resource/technical/document/datasheet/41/4f/b3/b0/12/d4/47/88/CD00000444.pdf/files/CD00000444.pdf/jcr:content/translations/en.CD00000444.pdf" H 1175 1450 50  0001 C CNN
 	1    1175 1500
@@
 F 0 "C301" H 850 2175 50  0000 L CNN
 F 1 "47U 25V" H 825 1975 50  0000 L CNN
-F 2 "" H 838 1925 50  0001 C CNN
+F 2 "Capacitors_THT:CP_Radial_D5.0mm_P2.50mm" H 838 1925 50  0001 C CNN
 F 3 "" H 800 2075 50  0001 C CNN
 	1    800  2075
@@
 F 0 "C302" H 1575 2125 50  0000 L CNN
 F 1 "22U" H 1575 1925 50  0000 L CNN
-F 2 "" H 1588 1875 50  0001 C CNN
+F 2 "Capacitors_THT:CP_Radial_D5.0mm_P2.50mm" H 1588 1875 50  0001 C CNN
 F 3 "" H 1550 2025 50  0001 C CNN
 	1    1550 2025
@@
 F 0 "R301" V 1825 1175 50  0000 L CNN
 F 1 "1K" H 1895 1230 50  0000 L CNN
-F 2 "" V 1755 1275 50  0001 C CNN
+F 2 "Resistors_ThroughHole:R_Axial_DIN0207_L6.3mm_D2.5mm_P7.62mm_Horizontal" V 1755 1275 50  0001 C CNN
 F 3 "" H 1825 1275 50  0001 C CNN
 	1    1825 1275
@@
 F 0 "R302" V 1825 2250 50  0000 L CNN
 F 1 "4K7" H 1895 2305 50  0000 L CNN
-F 2 "" V 1755 2350 50  0001 C CNN
+F 2 "Resistors_ThroughHole:R_Axial_DIN0207_L6.3mm_D2.5mm_P7.62mm_Horizontal" V 1755 2350 50  0001 C CNN
 F 3 "" H 1825 2350 50  0001 C CNN
 	1    1825 2350
@@
 F 0 "R303" H 4170 1121 50  0000 L CNN
 F 1 "100R" H 4170 1030 50  0000 L CNN
-F 2 "" V 4030 1075 50  0001 C CNN
+F 2 "Resistors_ThroughHole:R_Axial_DIN0207_L6.3mm_D2.5mm_P7.62mm_Horizontal" V 4030 1075 50  0001 C CNN
 F 3 "" H 4100 1075 50  0001 C CNN
 	1    4100 1075
@@
 F 0 "IC303" H 1175 1092 50  0000 C CNN
 F 1 "AZ1117-3.3" H 1175 1001 50  0000 C CNN
-F 2 "" H 1175 1100 50  0001 C CIN
+F 2 "TO_SOT_Packages_SMD:SOT-23_Handsoldering" H 1175 1100 50  0001 C CIN
 F 3 "https://www.diodes.com/assets/Datasheets/AZ1117.pdf" H 1175 850 50  0001 C CNN
 	1    1175 850
@@
 F 0 "J401" H 8993 2767 50  0000 C CNN
 F 1 "DB9_Male" H 8993 2676 50  0000 C CNN
-F 2 "" H 9075 2075 50  0001 C CNN
+F 2 "Connectors:DB9MC" H 9075 2075 50  0001 C CNN
 F 3 "" H 9075 2075 50  0001 C CNN
 	1    9075 2075
@@
 F 0 "R401" V 9500 1525 50  0000 L CNN
 F 1 "10K" V 9575 1550 50  0000 L CNN
-F 2 "" V 9430 1625 50  0001 C CNN
+F 2 "Resistors_ThroughHole:R_Axial_DIN0207_L6.3mm_D2.5mm_P7.62mm_Horizontal" V 9430 1625 50  0001 C CNN
 F 3 "" H 9500 1625 50  0001 C CNN
 	1    9500 1625
@@
 F 0 "IC501" H 9150 3150 50  0000 C CNN
 F 1 "YM2149" H 9650 3175 50  0000 C CNN
-F 2 "" H 9300 3775 50  0001 C CNN
+F 2 "Housings_DIP:DIP-40_W15.24mm_Socket_LongPads" H 9300 3775 50  0001 C CNN
 F 3 "" H 9300 3775 50  0001 C CNN
 	1    9400 4575
@@
 F 0 "J301" V 1800 3375 50  0000 L CNN
 F 1 "Conn_01x04" H 1755 3401 50  0001 L CNN
-F 2 "" H 1675 3500 50  0001 C CNN
+F 2 "Pin_Headers:Pin_Header_Straight_1x04_Pitch2.54mm" H 1675 3500 50  0001 C CNN
 F 3 "~" H 1675 3500 50  0001 C CNN
 	1    1675 3500
@@
 A0
 $Comp
-L Lattice:GAL16V8 UIC502
+L Lattice:GAL16V8 IC502
 U 1 1 5FC6FB56
 P 7325 5475
-F 0 "UIC502" H 7325 6291 50  0000 C CNN
+F 0 "IC502" H 7325 6291 50  0000 C CNN
 F 1 "GAL16V8" H 7325 6200 50  0000 C CNN
-F 2 "" H 7325 5475 50  0001 C CNN
+F 2 "Housings_DIP:DIP-20_W7.62mm_Socket_LongPads" H 7325 5475 50  0001 C CNN
 F 3 "" H 7325 5475 50  0001 C CNN
 	1    7325 5475
@@
 F 0 "J501" V 8125 5400 50  0000 L CNN
 F 1 "Conn_01x05" H 8105 5426 50  0001 L CNN
-F 2 "" H 8025 5475 50  0001 C CNN
+F 2 "Pin_Headers:Pin_Header_Straight_1x05_Pitch2.54mm" H 8025 5475 50  0001 C CNN
 F 3 "~" H 8025 5475 50  0001 C CNN
 	1    8025 5475
@@
 F 0 "J502" V 10300 4350 50  0000 L CNN
 F 1 "Conn_01x08" H 10280 4376 50  0001 L CNN
-F 2 "" H 10200 4475 50  0001 C CNN
+F 2 "Pin_Headers:Pin_Header_Straight_1x08_Pitch2.54mm" H 10200 4475 50  0001 C CNN
 F 3 "~" H 10200 4475 50  0001 C CNN
 	1    10200 4475
@@
 F 0 "J503" V 10325 5250 50  0000 L CNN
 F 1 "Conn_01x08" H 10280 5276 50  0001 L CNN
-F 2 "" H 10200 5375 50  0001 C CNN
+F 2 "Pin_Headers:Pin_Header_Straight_1x08_Pitch2.54mm" H 10200 5375 50  0001 C CNN
 F 3 "~" H 10200 5375 50  0001 C CNN
 	1    10200 5375
@@
 F 0 "R501" V 10150 3775 50  0000 C CNN
 F 1 "4K7" V 10100 3950 50  0000 C CNN
-F 2 "" V 10080 3775 50  0001 C CNN
+F 2 "Resistors_ThroughHole:R_Axial_DIN0207_L6.3mm_D2.5mm_P7.62mm_Horizontal" V 10080 3775 50  0001 C CNN
 F 3 "" H 10150 3775 50  0001 C CNN
 	1    10150 3775
@@
 F 0 "R502" V 10150 3875 50  0000 C CNN
 F 1 "4K7" V 10200 4050 50  0000 C CNN
-F 2 "" V 10080 3875 50  0001 C CNN
+F 2 "Resistors_ThroughHole:R_Axial_DIN0207_L6.3mm_D2.5mm_P7.62mm_Horizontal" V 10080 3875 50  0001 C CNN
 F 3 "" H 10150 3875 50  0001 C CNN
 	1    10150 3875
@@
 F 0 "R503" V 10150 3975 50  0000 C CNN
 F 1 "4K7" V 10000 4150 50  0000 C CNN
-F 2 "" V 10080 3975 50  0001 C CNN
+F 2 "Resistors_ThroughHole:R_Axial_DIN0207_L6.3mm_D2.5mm_P7.62mm_Horizontal" V 10080 3975 50  0001 C CNN
 F 3 "" H 10150 3975 50  0001 C CNN
 	1    10150 3975
@@
 F 0 "R504" H 10645 4071 50  0000 L CNN
 F 1 "1K" H 10645 3980 50  0000 L CNN
-F 2 "" V 10505 4025 50  0001 C CNN
+F 2 "Resistors_ThroughHole:R_Axial_DIN0207_L6.3mm_D2.5mm_P7.62mm_Horizontal" V 10505 4025 50  0001 C CNN
 F 3 "" H 10575 4025 50  0001 C CNN
 	1    10575 4025
@@
 F 0 "J504" V 7350 3900 50  0000 C CNN
 F 1 "Conn_01x07" H 7168 4301 50  0001 C CNN
-F 2 "" H 7250 3875 50  0001 C CNN
+F 2 "Pin_Headers:Pin_Header_Straight_1x07_Pitch2.54mm" H 7250 3875 50  0001 C CNN
 F 3 "~" H 7250 3875 50  0001 C CNN
 	1    7250 3875
@@
 F 0 "J601" H 5475 2400 50  0000 C CNN
 F 1 "Conn_02x08_Odd_Even" H 5475 2401 50  0001 C CNN
-F 2 "" H 5425 1975 50  0001 C CNN
+F 2 "Connectors:IDC_Header_Straight_16pins" H 5425 1975 50  0001 C CNN
 F 3 "~" H 5425 1975 50  0001 C CNN
 	1    5425 1975
@@
 F 0 "J701" H 7175 3200 50  0000 C CNN
 F 1 "Conn_02x23_Row_Letter_First" H 7175 3201 50  0001 C CNN
-F 2 "" H 7125 1975 50  0001 C CNN
+F 2 "Pin_Headers:Pin_Header_Straight_2x23_Pitch2.54mm" H 7125 1975 50  0001 C CNN
 F 3 "~" H 7125 1975 50  0001 C CNN
 	1    7125 1975
@@
 F 0 "J702" V 8450 2525 50  0000 L CNN
 F 1 "Conn_01x09" H 8430 2576 50  0001 L CNN
-F 2 "" H 8350 2625 50  0001 C CNN
+F 2 "Pin_Headers:Pin_Header_Straight_1x09_Pitch2.54mm" H 8350 2625 50  0001 C CNN
 F 3 "~" H 8350 2625 50  0001 C CNN
 	1    8350 2625
@@
 F 0 "J703" V 8450 1575 50  0000 L CNN
 F 1 "Conn_01x09" H 8430 1651 50  0001 L CNN
-F 2 "" H 8350 1700 50  0001 C CNN
+F 2 "Pin_Headers:Pin_Header_Straight_1x09_Pitch2.54mm" H 8350 1700 50  0001 C CNN
 F 3 "~" H 8350 1700 50  0001 C CNN
 	1    8350 1700

Commit message: Added mounring holes
Parts:
- J701: footprint Pin_Headers:Pin_Header_Straight_2x23_Pitch2.54mm -> zxbus:Pin_Header_Straight_2x23_Pitch2.54mm
Changed lines of the file:
@@
 F 0 "J701" H 7175 3200 50  0000 C CNN
 F 1 "Conn_02x23_Row_Letter_First" H 7175 3201 50  0001 C CNN
-F 2 "Pin_Headers:Pin_Header_Straight_2x23_Pitch2.54mm" H 7125 1975 50  0001 C CNN
+F 2 "zxbus:Pin_Header_Straight_2x23_Pitch2.54mm" H 7125 1975 50  0001 C CNN
 F 3 "~" H 7125 1975 50  0001 C CNN
 	1    7125 1975

Commit message: Placement getting there
Parts:
- added C303: 10N, Capacitors_SMD:C_0603_HandSoldering, symbol device:C
- added IC801: AS6C4008Extra, zxbus:DIP-4_W15.24mm_Socket_LongPads, symbol zxbus:AS6C4008Extra
- renumbered QTR403 to TR403
Connections:
- net labels added: +3V3
- wire segments 88 -> 96
Changed lines of the file:
@@
 	1475 850  1475 1500
 Connection ~ 1475 1500
-Wire Wire Line
-	875  850  875  1500
-Connection ~ 875  1500
 $Comp
 L power:GND #PWR0133
 U 1 1 6327B84A
-P 1175 1150
-F 0 "#PWR0133" H 1175 900 50  0001 C CNN
-F 1 "GND" V 1180 1022 50  0000 R CNN
-F 2 "" H 1175 1150 50  0001 C CNN
-F 3 "" H 1175 1150 50  0001 C CNN
-	1    1175 1150
+P 675 1150
+F 0 "#PWR0133" H 675 900 50  0001 C CNN
+F 1 "GND" V 550 1100 50  0000 R CNN
+F 2 "" H 675 1150 50  0001 C CNN
+F 3 "" H 675 1150 50  0001 C CNN
+	1    675  1150
 	0    1    1    0
 $EndComp
@@
 $EndComp
 $Comp
-L Transistor:2N3904 QTR403
+L Transistor:2N3904 TR403
 U 1 1 633427C1
 P 10275 1925
-F 0 "QTR403" H 10465 1971 50  0000 L CNN
+F 0 "TR403" H 10465 1971 50  0000 L CNN
 F 1 "2N3904" H 10465 1880 50  0000 L CNN
 F 2 "TO_SOT_Packages_THT:TO-92_Molded_Narrow" H 10475 1850 50  0001 L CIN
@@
 A8'
 NoConn ~ 2100 1600
+$Comp
+L power:+3V3 #PWR0151
+U 1 1 5FD19FCC
+P 1550 1500
+F 0 "#PWR0151" H 1550 1350 50  0001 C CNN
+F 1 "+3V3" H 1565 1673 50  0000 C CNN
+F 2 "" H 1550 1500 50  0001 C CNN
+F 3 "" H 1550 1500 50  0001 C CNN
+	1    1550 1500
+	1    0    0    -1
+$EndComp
+$Comp
+L power:+5V #PWR0152
+U 1 1 5FD1EBA5
+P 650 850
+F 0 "#PWR0152" H 650 700 50  0001 C CNN
+F 1 "+5V" V 725 850 50  0000 L CNN
+F 2 "" H 650 850 50  0001 C CNN
+F 3 "" H 650 850 50  0001 C CNN
+	1    650  850
+	0    -1   -1   0
+$EndComp
+Wire Wire Line
+	875  850  725  850
+$Comp
+L device:C C303
+U 1 1 5FD2207C
+P 725 1000
+F 0 "C303" H 750 1100 50  0000 L CNN
+F 1 "10N" H 775 900 50  0000 L CNN
+F 2 "Capacitors_SMD:C_0603_HandSoldering" H 763 850 50  0001 C CNN
+F 3 "" H 725 1000 50  0001 C CNN
+	1    725  1000
+	1    0    0    -1
+$EndComp
+Connection ~ 725  850
+Wire Wire Line
+	725  850  650  850
+Wire Wire Line
+	1175 1150 725  1150
+Wire Wire Line
+	725  1150 675  1150
+Connection ~ 725  1150
+$Comp
+L zxbus:AS6C4008Extra IC801
+U 1 1 5FDF782D
+P 5850 8100
+F 0 "IC801" H 5850 9117 50  0000 C CNN
+F 1 "AS6C4008Extra" H 5850 9026 50  0000 C CNN
+F 2 "zxbus:DIP-4_W15.24mm_Socket_LongPads" H 5850 8100 50  0001 C CIN
+F 3 "" H 5850 8100 50  0001 C CNN
+	1    5850 8100
+	1    0    0    -1
+$EndComp
+$Comp
+L power:+5V #PWR0153
+U 1 1 5FDF89AC
+P 6425 7300
+F 0 "#PWR0153" H 6425 7150 50  0001 C CNN
+F 1 "+5V" H 6440 7473 50  0000 C CNN
+F 2 "" H 6425 7300 50  0001 C CNN
+F 3 "" H 6425 7300 50  0001 C CNN
+	1    6425 7300
+	1    0    0    -1
+$EndComp
+Wire Wire Line
+	6425 7300 6425 7350
+Wire Wire Line
+	6425 7350 6350 7350
+Text GLabel 6350 7450 2    50   Input ~ 0
+A15
+Wire Wire Line
+	5350 7350 5250 7350
+Wire Wire Line
+	5250 7350 5250 7450
+Wire Wire Line
+	5250 7450 5350 7450
+Text GLabel 5250 7400 0    50   Input ~ 0
+A14
 $EndSCHEMATC
