File: KiCad/ZX21/ZX21_Extras.sch (KiCad schematic (older format))
At the start: 32 parts, among them IC301 3V3 PSU, IC302 ESP32-WROOM, IC303 AZ1117-3.3, IC501 YM2149, IC502 GAL16V8, IC801 AS6C4008Extra, J301 Conn_01x04, J401 DB9_Male, J501 Conn_01x06, J502 Conn_01x08, J503 Conn_01x08, J504 Conn_01x07, J601 Conn_02x08_Odd_Even, J701 Conn_02x23_Row_Letter_First, J702 Conn_01x09, J703 Conn_01x09

Commit message: Added option for YMZ284 :D
Parts:
- removed J504: Conn_01x07, Pin_Headers:Pin_Header_Straight_1x07_Pitch2.54mm, symbol Connector:Conn_01x07
- added C501: 100N, Capacitors_THT:C_Disc_D4.7mm_W2.5mm_P5.00mm, symbol device:C
- added IC503: YMZ284, Housings_DIP:DIP-16_W7.62mm_Socket_LongPads, symbol Sinclair:YMZ284
- added J302: Conn_01x03, Pin_Headers:Pin_Header_Straight_1x03_Pitch2.54mm, symbol Connector:Conn_01x03
- added J504: Conn_01x08, Pin_Headers:Pin_Header_Straight_1x08_Pitch2.54mm, symbol Connector:Conn_01x08
Connections:
- wire segments 93 -> 108
- no-connect marks 39 -> 37
Other:
- moved on the sheet: J401, J601, J701, J702, J703, R401, TR401, TR402, TR403, TR404, TR405

Commit message: Fixing DRC Issues
Parts:
- C301, C302: footprint Capacitors_THT:CP_Radial_D5.0mm_P2.50mm -> Capacitors_ThroughHole:CP_Radial_D5.0mm_P2.50mm
- C501: footprint Capacitors_THT:C_Disc_D4.7mm_W2.5mm_P5.00mm -> Capacitors_ThroughHole:C_Disc_D4.7mm_W2.5mm_P5.00mm
- R301, R302, R303, R401, R501, R502, R503, R504: footprint Resistors_ThroughHole:R_Axial_DIN0207_L6.3mm_D2.5mm_P7.62mm_Horizontal -> Resistors_ThroughHole:R_Axial_DIN0204_L3.6mm_D1.6mm_P7.62mm_Horizontal
Changed lines of the file:
@@
 F 0 "C301" H 850 2175 50  0000 L CNN
 F 1 "47U 25V" H 825 1975 50  0000 L CNN
-F 2 "Capacitors_THT:CP_Radial_D5.0mm_P2.50mm" H 838 1925 50  0001 C CNN
+F 2 "Capacitors_ThroughHole:CP_Radial_D5.0mm_P2.50mm" H 838 1925 50  0001 C CNN
 F 3 "" H 800 2075 50  0001 C CNN
 	1    800  2075
@@
 F 0 "C302" H 1575 2125 50  0000 L CNN
 F 1 "22U" H 1575 1925 50  0000 L CNN
-F 2 "Capacitors_THT:CP_Radial_D5.0mm_P2.50mm" H 1588 1875 50  0001 C CNN
+F 2 "Capacitors_ThroughHole:CP_Radial_D5.0mm_P2.50mm" H 1588 1875 50  0001 C CNN
 F 3 "" H 1550 2025 50  0001 C CNN
 	1    1550 2025
@@
 F 0 "R301" V 1825 1175 50  0000 L CNN
 F 1 "1K" H 1895 1230 50  0000 L CNN
-F 2 "Resistors_ThroughHole:R_Axial_DIN0207_L6.3mm_D2.5mm_P7.62mm_Horizontal" V 1755 1275 50  0001 C CNN
+F 2 "Resistors_ThroughHole:R_Axial_DIN0204_L3.6mm_D1.6mm_P7.62mm_Horizontal" V 1755 1275 50  0001 C CNN
 F 3 "" H 1825 1275 50  0001 C CNN
 	1    1825 1275
@@
 F 0 "R302" V 1825 2250 50  0000 L CNN
 F 1 "4K7" H 1895 2305 50  0000 L CNN
-F 2 "Resistors_ThroughHole:R_Axial_DIN0207_L6.3mm_D2.5mm_P7.62mm_Horizontal" V 1755 2350 50  0001 C CNN
+F 2 "Resistors_ThroughHole:R_Axial_DIN0204_L3.6mm_D1.6mm_P7.62mm_Horizontal" V 1755 2350 50  0001 C CNN
 F 3 "" H 1825 2350 50  0001 C CNN
 	1    1825 2350
@@
 F 0 "R303" H 4170 1121 50  0000 L CNN
 F 1 "100R" H 4170 1030 50  0000 L CNN
-F 2 "Resistors_ThroughHole:R_Axial_DIN0207_L6.3mm_D2.5mm_P7.62mm_Horizontal" V 4030 1075 50  0001 C CNN
+F 2 "Resistors_ThroughHole:R_Axial_DIN0204_L3.6mm_D1.6mm_P7.62mm_Horizontal" V 4030 1075 50  0001 C CNN
 F 3 "" H 4100 1075 50  0001 C CNN
 	1    4100 1075
@@
 F 0 "R401" V 5625 1650 50  0000 L CNN
 F 1 "10K" V 5700 1675 50  0000 L CNN
-F 2 "Resistors_ThroughHole:R_Axial_DIN0207_L6.3mm_D2.5mm_P7.62mm_Horizontal" V 5555 1750 50  0001 C CNN
+F 2 "Resistors_ThroughHole:R_Axial_DIN0204_L3.6mm_D1.6mm_P7.62mm_Horizontal" V 5555 1750 50  0001 C CNN
 F 3 "" H 5625 1750 50  0001 C CNN
 	1    5625 1750
@@
 F 0 "R502" V 10150 3875 50  0000 C CNN
 F 1 "4K7" V 10200 4050 50  0000 C CNN
-F 2 "Resistors_ThroughHole:R_Axial_DIN0207_L6.3mm_D2.5mm_P7.62mm_Horizontal" V 10080 3875 50  0001 C CNN
+F 2 "Resistors_ThroughHole:R_Axial_DIN0204_L3.6mm_D1.6mm_P7.62mm_Horizontal" V 10080 3875 50  0001 C CNN
 F 3 "" H 10150 3875 50  0001 C CNN
 	1    10150 3875
@@
 F 0 "R503" V 10150 3975 50  0000 C CNN
 F 1 "4K7" V 10000 4150 50  0000 C CNN
-F 2 "Resistors_ThroughHole:R_Axial_DIN0207_L6.3mm_D2.5mm_P7.62mm_Horizontal" V 10080 3975 50  0001 C CNN
+F 2 "Resistors_ThroughHole:R_Axial_DIN0204_L3.6mm_D1.6mm_P7.62mm_Horizontal" V 10080 3975 50  0001 C CNN
 F 3 "" H 10150 3975 50  0001 C CNN
 	1    10150 3975
@@
 F 0 "R504" H 10645 4071 50  0000 L CNN
 F 1 "1K" H 10645 3980 50  0000 L CNN
-F 2 "Resistors_ThroughHole:R_Axial_DIN0207_L6.3mm_D2.5mm_P7.62mm_Horizontal" V 10505 4025 50  0001 C CNN
+F 2 "Resistors_ThroughHole:R_Axial_DIN0204_L3.6mm_D1.6mm_P7.62mm_Horizontal" V 10505 4025 50  0001 C CNN
 F 3 "" H 10575 4025 50  0001 C CNN
 	1    10575 4025
@@
 F 0 "R501" V 10150 3775 50  0000 C CNN
 F 1 "4K7" V 10100 3950 50  0000 C CNN
-F 2 "Resistors_ThroughHole:R_Axial_DIN0207_L6.3mm_D2.5mm_P7.62mm_Horizontal" V 10080 3775 50  0001 C CNN
+F 2 "Resistors_ThroughHole:R_Axial_DIN0204_L3.6mm_D1.6mm_P7.62mm_Horizontal" V 10080 3775 50  0001 C CNN
 F 3 "" H 10150 3775 50  0001 C CNN
 	1    10150 3775
@@
 F 0 "C501" H 10415 2971 50  0000 L CNN
 F 1 "100N" H 10415 2880 50  0000 L CNN
-F 2 "Capacitors_THT:C_Disc_D4.7mm_W2.5mm_P5.00mm" H 10338 2775 50  0001 C CNN
+F 2 "Capacitors_ThroughHole:C_Disc_D4.7mm_W2.5mm_P5.00mm" H 10338 2775 50  0001 C CNN
 F 3 "" H 10300 2925 50  0001 C CNN
 	1    10300 2925

Commit message: Fixing DRC Issues
Parts:
- J502, J503, J504: footprint Pin_Headers:Pin_Header_Straight_1x08_Pitch2.54mm -> zxbus:Pin_Header_Straight_1x08_Pitch2.54mm
Changed lines of the file:
@@
 F 0 "J502" V 10300 4350 50  0000 L CNN
 F 1 "Conn_01x08" H 10280 4376 50  0001 L CNN
-F 2 "Pin_Headers:Pin_Header_Straight_1x08_Pitch2.54mm" H 10200 4475 50  0001 C CNN
+F 2 "zxbus:Pin_Header_Straight_1x08_Pitch2.54mm" H 10200 4475 50  0001 C CNN
 F 3 "~" H 10200 4475 50  0001 C CNN
 	1    10200 4475
@@
 F 0 "J503" V 10325 5250 50  0000 L CNN
 F 1 "Conn_01x08" H 10280 5276 50  0001 L CNN
-F 2 "Pin_Headers:Pin_Header_Straight_1x08_Pitch2.54mm" H 10200 5375 50  0001 C CNN
+F 2 "zxbus:Pin_Header_Straight_1x08_Pitch2.54mm" H 10200 5375 50  0001 C CNN
 F 3 "~" H 10200 5375 50  0001 C CNN
 	1    10200 5375
@@
 F 0 "J504" H 7750 4525 50  0000 C CNN
 F 1 "Conn_01x08" H 7618 4551 50  0001 C CNN
-F 2 "Pin_Headers:Pin_Header_Straight_1x08_Pitch2.54mm" H 7700 4125 50  0001 C CNN
+F 2 "zxbus:Pin_Header_Straight_1x08_Pitch2.54mm" H 7700 4125 50  0001 C CNN
 F 3 "~" H 7700 4125 50  0001 C CNN
 	1    7700 4125

Commit message: FIrst go at DRC complete
Parts:
- J302: footprint Pin_Headers:Pin_Header_Straight_1x03_Pitch2.54mm -> zxbus:Pin_Header_Straight_1x03_Pitch2.54mm
Changed lines of the file:
@@
 F 0 "J302" H 4275 1425 50  0000 L CNN
 F 1 "Conn_01x03" H 4455 1601 50  0001 L CNN
-F 2 "Pin_Headers:Pin_Header_Straight_1x03_Pitch2.54mm" H 4375 1650 50  0001 C CNN
+F 2 "zxbus:Pin_Header_Straight_1x03_Pitch2.54mm" H 4375 1650 50  0001 C CNN
 F 3 "~" H 4375 1650 50  0001 C CNN
 	1    4375 1650

Commit message: ESP32 Flipped
Parts:
- IC301: footprint TO_SOT_Packages_THT:TO-220-3_Horizontal -> TO_SOT_Packages_THT:TO-220-3_Vertical
Changed lines of the file:
@@
 F 0 "IC301" H 1175 1742 50  0000 C CNN
 F 1 "3V3 PSU" H 1175 1651 50  0000 C CNN
-F 2 "TO_SOT_Packages_THT:TO-220-3_Horizontal" H 1200 1350 50  0001 L CIN
+F 2 "TO_SOT_Packages_THT:TO-220-3_Vertical" H 1200 1350 50  0001 L CIN
 F 3 "http://www.st.com/content/ccc/resource/technical/document/datasheet/41/4f/b3/b0/12/d4/47/88/CD00000444.pdf/files/CD00000444.pdf/jcr:content/translations/en.CD00000444.pdf" H 1175 1450 50  0001 C CNN
 	1    1175 1500
